File: Hardware/LoRa Photon 2 PCB/LoRa_Photon2/LoRa_Photon2.sch (EAGLE design)
At the start: 24 parts, among them IC1 74HC14N, U1 PHOTON2

Commit message: Added Photon 2 PCB
Added Eagle files, schematic pdf and rendering of the board to the Hardware folder.
Parts:
- renumbered GRN-D9 to GRN, RED-D8 to RED
Changed lines of the file:
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@@
 </classes>
 <parts>
-<part name="GRN-D9" library="led" library_urn="urn:adsk.eagle:library:259" deviceset="TLLG4400" device="" package3d_urn="urn:adsk.eagle:package:15797/1"/>
-<part name="RED-D8" library="led" library_urn="urn:adsk.eagle:library:259" deviceset="TLLR4400" device="" package3d_urn="urn:adsk.eagle:package:15797/1"/>
+<part name="GRN" library="led" library_urn="urn:adsk.eagle:library:259" deviceset="TLLG4400" device="" package3d_urn="urn:adsk.eagle:package:15797/1"/>
+<part name="RED" library="led" library_urn="urn:adsk.eagle:library:259" deviceset="TLLR4400" device="" package3d_urn="urn:adsk.eagle:package:15797/1"/>
 <part name="CONTACT_SENSOR" library="SparkFun-Connectors" library_urn="urn:adsk.eagle:library:513" deviceset="CONN_02" device="3.5MM" package3d_urn="urn:adsk.eagle:package:38050/1"/>
 <part name="DIGITAL/ANALOG" library="con-lstb" library_urn="urn:adsk.eagle:library:162" deviceset="MA08-1" device="" package3d_urn="urn:adsk.eagle:package:8343/1"/>
@@
 </plain>
 <instances>
-<instance part="GRN-D9" gate="G$1" x="104.14" y="78.74" smashed="yes">
+<instance part="GRN" gate="G$1" x="104.14" y="78.74" smashed="yes">
 <attribute name="NAME" x="107.696" y="74.168" size="1.778" layer="95" rot="R90"/>
 <attribute name="VALUE" x="109.855" y="74.168" size="1.778" layer="96" rot="R90"/>
 </instance>
-<instance part="RED-D8" gate="G$1" x="-10.16" y="86.36" smashed="yes">
+<instance part="RED" gate="G$1" x="-10.16" y="86.36" smashed="yes">
 <attribute name="NAME" x="-6.604" y="81.788" size="1.778" layer="95" rot="R90"/>
 <attribute name="VALUE" x="-4.445" y="81.788" size="1.778" layer="96" rot="R90"/>
@@
 </segment>
 <segment>
-<pinref part="GRN-D9" gate="G$1" pin="C"/>
+<pinref part="GRN" gate="G$1" pin="C"/>
 <pinref part="SUPPLY4" gate="GND" pin="GND"/>
 <wire x1="104.14" y1="73.66" x2="104.14" y2="66.04" width="0.1524" layer="91"/>
 </segment>
 <segment>
-<pinref part="RED-D8" gate="G$1" pin="C"/>
+<pinref part="RED" gate="G$1" pin="C"/>
 <pinref part="SUPPLY5" gate="GND" pin="GND"/>
 <wire x1="-10.16" y1="81.28" x2="-10.16" y2="78.74" width="0.1524" layer="91"/>
@@
 <segment>
 <pinref part="R1" gate="G$1" pin="1"/>
-<pinref part="RED-D8" gate="G$1" pin="A"/>
+<pinref part="RED" gate="G$1" pin="A"/>
 <wire x1="-10.16" y1="88.9" x2="-10.16" y2="96.52" width="0.1524" layer="91"/>
 </segment>
@@
 <segment>
 <pinref part="R2" gate="G$1" pin="1"/>
-<pinref part="GRN-D9" gate="G$1" pin="A"/>
+<pinref part="GRN" gate="G$1" pin="A"/>
 <wire x1="104.14" y1="86.36" x2="104.14" y2="81.28" width="0.1524" layer="91"/>
 </segment>

Commit message: Minor changes to schematic
Only changed labels on schematic.  Does not alter the netlist or the board layout.
Other:
- note added: "SCLK"
- note removed: "!SS"
Changed lines of the file:
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@@
 <text x="134.62" y="93.98" size="1.778" layer="91">GND</text>
 <text x="134.62" y="91.44" size="1.778" layer="91">GND</text>
-<text x="86.36" y="71.12" size="1.778" layer="91">MISO</text>
-<text x="86.36" y="73.66" size="1.778" layer="91">MOSI</text>
-<text x="86.36" y="76.2" size="1.778" layer="91">!SS</text>
+<text x="86.36" y="71.12" size="1.778" layer="91">S3</text>
+<text x="86.36" y="73.66" size="1.778" layer="91">SCLK</text>
+<text x="86.36" y="76.2" size="1.778" layer="91">MOSI</text>
 <text x="86.36" y="83.82" size="1.778" layer="91">VCC</text>
 <text x="86.36" y="81.28" size="1.778" layer="91">VCC</text>
-<text x="86.36" y="78.74" size="1.778" layer="91">S3</text>
+<text x="86.36" y="78.74" size="1.778" layer="91">MISO</text>
 <text x="86.36" y="68.58" size="1.778" layer="91">GND</text>
 <text x="86.36" y="66.04" size="1.778" layer="91">GND</text>
